File: Pedales/Pedales.kicad_pcb (KiCad board)
At the start: 2 copper layers, 23 parts, among them J1 IN, J2 9V, J3 OUT, U1 opamp

Commit message: Add files via upload
Other:
- board outline added: 29.1 x 23.7 mm
Changed lines of the file:
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@@
       (net 23 "/9V") (pinfunction "1") (pintype "passive"))
   )
+  (gr_rect (start 97.45 85.2) (end 126.55 108.9) (layer "Edge.Cuts") (width 0.1) (fill none))
   (segment (start 106.55 104.45) (end 106.6 104.4) (width 0.25) (layer "F.Cu") (net 1))
   (segment (start 106.6 103.55) (end 106.6 104.4) (width 0.25) (layer "F.Cu") (net 1))
