File: Pedales/Pedales.kicad_sch (KiCad schematic)
At the start: 23 parts, among them J1 IN, J2 9V, J3 OUT, U1 opamp

Commit message: Add files via upload
Other:
- title: (none) -> Guitar effects template by Ariel Robotti
Changed lines of the file:
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@@
 (kicad_sch (version 20211123) (generator eeschema)
   (paper "A4")
+  (title_block
+    (title "Guitar effects template by Ariel Robotti")
+    (date "2022-06-30")
+  )
   (junction (at 127 78.74) (diameter 0) (color 0 0 0 0)
   )
